File: vna-steps/slowdds/dds.sch (KiCad schematic (older format))
At the start: 5 parts

Commit message: slowdds layout completed. images + schematics generated. ZIP file scripts added and documented in README. slowdds gerbers generated + zipped.
Parts:
- C10, C11: renamed from C?; footprint (none) -> Capacitors_SMD:C_0402
- TP4, TP5: renamed from TP?; footprint MODULE -> bce:TP
- U5: renamed from U?; footprint MODULE -> Housings_SSOP:MSOP-10_3x3mm_Pitch0.5mm
Changed lines of the file:
@@
 $EndDescr
 $Comp
-L AD9833 U?
+L AD9833 U5
 U 1 1 558544D6
 P 6050 4050
-F 0 "U?" H 6050 3950 50  0000 C CNN
+F 0 "U5" H 6050 3950 50  0000 C CNN
 F 1 "AD9833" H 6050 4150 50  0000 C CNN
-F 2 "MODULE" H 6050 4350 50  0001 C CNN
+F 2 "Housings_SSOP:MSOP-10_3x3mm_Pitch0.5mm" H 6050 4350 50  0001 C CNN
 F 3 "DOCUMENTATION" H 6050 3750 50  0001 C CNN
 	1    6050 4050
@@
 $EndComp
 $Comp
-L C C?
+L C C10
 U 1 1 558545DE
 P 4750 4200
-F 0 "C?" H 4775 4300 50  0000 L CNN
+F 0 "C10" H 4775 4300 50  0000 L CNN
 F 1 "100n" H 4775 4100 50  0000 L CNN
-F 2 "" H 4788 4050 30  0000 C CNN
+F 2 "Capacitors_SMD:C_0402" H 4788 4050 30  0001 C CNN
 F 3 "" H 4750 4200 60  0000 C CNN
 	1    4750 4200
@@
 $EndComp
 $Comp
-L GND #PWR?
+L GND #PWR031
 U 1 1 55854617
 P 4750 4350
-F 0 "#PWR?" H 4750 4100 50  0001 C CNN
+F 0 "#PWR031" H 4750 4100 50  0001 C CNN
 F 1 "GND" H 4750 4200 50  0000 C CNN
 F 2 "" H 4750 4350 60  0000 C CNN
@@
 $EndComp
 $Comp
-L GND #PWR?
+L GND #PWR032
 U 1 1 5585462D
 P 5000 4250
-F 0 "#PWR?" H 5000 4000 50  0001 C CNN
+F 0 "#PWR032" H 5000 4000 50  0001 C CNN
 F 1 "GND" H 5000 4100 50  0000 C CNN
 F 2 "" H 5000 4250 60  0000 C CNN
@@
 	7000 3850 6800 3850
 $Comp
-L GND #PWR?
+L GND #PWR033
 U 1 1 55854706
 P 7500 4050
-F 0 "#PWR?" H 7500 3800 50  0001 C CNN
+F 0 "#PWR033" H 7500 3800 50  0001 C CNN
 F 1 "GND" H 7500 3900 50  0000 C CNN
 F 2 "" H 7500 4050 60  0000 C CNN
@@
 	7500 3950 7500 4050
 $Comp
-L +3.3VDAC #PWR?
+L +3.3VDAC #PWR034
 U 1 1 5585473D
 P 4800 3950
-F 0 "#PWR?" H 4950 3900 50  0001 C CNN
+F 0 "#PWR034" H 4950 3900 50  0001 C CNN
 F 1 "+3.3VDAC" H 4800 4050 50  0000 C CNN
 F 2 "" H 4800 3950 60  0000 C CNN
@@
 	4800 3950 5300 3950
 $Comp
-L C C?
+L C C11
 U 1 1 55854763
 P 5000 3800
-F 0 "C?" H 5025 3900 50  0000 L CNN
+F 0 "C11" H 5025 3900 50  0000 L CNN
 F 1 "10n" H 5025 3700 50  0000 L CNN
-F 2 "" H 5038 3650 30  0000 C CNN
+F 2 "Capacitors_SMD:C_0402" H 5038 3650 30  0001 C CNN
 F 3 "" H 5000 3800 60  0000 C CNN
 	1    5000 3800
@@
 Connection ~ 5000 3950
 $Comp
-L TP TP?
+L TP TP4
 U 1 1 558547B9
 P 6050 4900
-F 0 "TP?" H 6050 4800 50  0000 C CNN
+F 0 "TP4" H 6050 4800 50  0000 C CNN
 F 1 "25MHz" H 6050 5000 50  0000 C CNN
-F 2 "MODULE" H 5800 4750 50  0001 C CNN
+F 2 "bce:TP" H 5800 4750 50  0001 C CNN
 F 3 "DOCUMENTATION" H 6050 4900 50  0001 C CNN
 	1    6050 4900
@@
 $EndComp
 $Comp
-L TP TP?
+L TP TP5
 U 1 1 55854804
 P 7800 3450
-F 0 "TP?" H 7800 3350 50  0000 C CNN
+F 0 "TP5" H 7800 3350 50  0000 C CNN
 F 1 "DDSOUT" H 7800 3550 50  0000 C CNN
-F 2 "MODULE" H 7550 3300 50  0001 C CNN
+F 2 "bce:TP" H 7550 3300 50  0001 C CNN
 F 3 "DOCUMENTATION" H 7800 3450 50  0001 C CNN
 	1    7800 3450
