File: vna-steps/slowdds/mcu.sch (KiCad schematic (older format))
At the start: 5 parts

Commit message: slowdds layout completed. images + schematics generated. ZIP file scripts added and documented in README. slowdds gerbers generated + zipped.
Parts:
- C8, C9: renamed from C?; footprint (none) -> Capacitors_SMD:C_0402
- R5, R6: renamed from R?; footprint (none) -> Resistors_SMD:R_0402
- U4: renamed from U?; footprint MODULE -> Housings_SSOP:TSSOP-20_4.4x6.5mm_Pitch0.65mm
Connections:
- net +3V3: now also C8.1, R5.1, U4.5 (VDDA)
Changed lines of the file:
@@
 $EndDescr
 $Comp
-L STM32F030F4 U?
+L STM32F030F4 U4
 U 1 1 55852DAB
 P 5750 3300
-F 0 "U?" H 5750 3000 50  0000 C CNN
+F 0 "U4" H 5750 3000 50  0000 C CNN
 F 1 "STM32F030F4" H 5750 3100 50  0000 C CNN
-F 2 "MODULE" H 5750 2750 50  0001 C CNN
+F 2 "Housings_SSOP:TSSOP-20_4.4x6.5mm_Pitch0.65mm" H 5750 2750 50  0001 C CNN
 F 3 "DOCUMENTATION" H 5750 3850 50  0001 C CNN
 	1    5750 3300
@@
 $EndComp
 $Comp
-L R R?
+L R R6
 U 1 1 55852E59
 P 4800 2550
-F 0 "R?" V 4880 2550 50  0000 C CNN
+F 0 "R6" V 4880 2550 50  0000 C CNN
 F 1 "10k" V 4800 2550 50  0000 C CNN
-F 2 "" V 4730 2550 30  0000 C CNN
+F 2 "Resistors_SMD:R_0402" V 4730 2550 30  0001 C CNN
 F 3 "" H 4800 2550 30  0000 C CNN
 	1    4800 2550
@@
 $EndComp
 $Comp
-L GND #PWR?
+L GND #PWR025
 U 1 1 55852E84
 P 4800 2700
-F 0 "#PWR?" H 4800 2450 50  0001 C CNN
+F 0 "#PWR025" H 4800 2450 50  0001 C CNN
 F 1 "GND" H 4800 2550 50  0000 C CNN
 F 2 "" H 4800 2700 60  0000 C CNN
@@
 $EndComp
 $Comp
-L R R?
+L R R5
 U 1 1 55852F2A
 P 4350 3000
-F 0 "R?" V 4430 3000 50  0000 C CNN
+F 0 "R5" V 4430 3000 50  0000 C CNN
 F 1 "10k" V 4350 3000 50  0000 C CNN
-F 2 "" V 4280 3000 30  0000 C CNN
+F 2 "Resistors_SMD:R_0402" V 4280 3000 30  0001 C CNN
 F 3 "" H 4350 3000 30  0000 C CNN
 	1    4350 3000
@@
 	4850 2950 5000 2950
 $Comp
-L C C?
+L C C8
 U 1 1 55852FCE
 P 4100 3400
-F 0 "C?" H 4125 3500 50  0000 L CNN
+F 0 "C8" H 4125 3500 50  0000 L CNN
 F 1 "100n" H 4125 3300 50  0000 L CNN
-F 2 "" H 4138 3250 30  0000 C CNN
+F 2 "Capacitors_SMD:C_0402" H 4138 3250 30  0001 C CNN
 F 3 "" H 4100 3400 60  0000 C CNN
 	1    4100 3400
@@
 	4100 3250 5000 3250
 $Comp
-L C C?
+L C C9
 U 1 1 55853006
 P 7250 3400
-F 0 "C?" H 7275 3500 50  0000 L CNN
+F 0 "C9" H 7275 3500 50  0000 L CNN
 F 1 "100n" H 7275 3300 50  0000 L CNN
-F 2 "" H 7288 3250 30  0000 C CNN
+F 2 "Capacitors_SMD:C_0402" H 7288 3250 30  0001 C CNN
 F 3 "" H 7250 3400 60  0000 C CNN
 	1    7250 3400
@@
 $EndComp
 Wire Wire Line
-	6500 3250 7150 3250
-Wire Wire Line
-	7150 3250 7250 3250
+	6500 3250 7250 3250
 $Comp
-L GND #PWR?
+L GND #PWR026
 U 1 1 5585309D
 P 7250 3550
-F 0 "#PWR?" H 7250 3300 50  0001 C CNN
+F 0 "#PWR026" H 7250 3300 50  0001 C CNN
 F 1 "GND" H 7250 3400 50  0000 C CNN
 F 2 "" H 7250 3550 60  0000 C CNN
@@
 	7050 3550 7250 3550
 $Comp
-L GND #PWR?
+L GND #PWR027
 U 1 1 558530C2
 P 4100 3550
-F 0 "#PWR?" H 4100 3300 50  0001 C CNN
+F 0 "#PWR027" H 4100 3300 50  0001 C CNN
 F 1 "GND" H 4100 3400 50  0000 C CNN
 F 2 "" H 4100 3550 60  0000 C CNN
@@
 $EndComp
 $Comp
-L +3.3V #PWR?
+L +3.3V #PWR028
 U 1 1 5585312F
 P 7150 3250
-F 0 "#PWR?" H 7150 3100 50  0001 C CNN
+F 0 "#PWR028" H 7150 3100 50  0001 C CNN
 F 1 "+3.3V" H 7150 3390 50  0000 C CNN
 F 2 "" H 7150 3250 60  0000 C CNN
@@
 Connection ~ 7150 3250
 $Comp
-L +3.3V #PWR?
+L +3.3V #PWR029
 U 1 1 5585314D
-P 4350 2900
-F 0 "#PWR?" H 4350 2750 50  0001 C CNN
-F 1 "+3.3V" H 4350 3040 50  0000 C CNN
-F 2 "" H 4350 2900 60  0000 C CNN
-F 3 "" H 4350 2900 60  0000 C CNN
-	1    4350 2900
+P 4350 2850
+F 0 "#PWR029" H 4350 2700 50  0001 C CNN
+F 1 "+3.3V" H 4350 2990 50  0000 C CNN
+F 2 "" H 4350 2850 60  0000 C CNN
+F 3 "" H 4350 2850 60  0000 C CNN
+	1    4350 2850
 	1    0    0    -1
 $EndComp
@@
 NoConn ~ 5000 3350
 NoConn ~ 5000 3450
+$Comp
+L +3.3V #PWR030
+U 1 1 55856D53
+P 4100 3250
+F 0 "#PWR030" H 4100 3100 50  0001 C CNN
+F 1 "+3.3V" H 4100 3390 50  0000 C CNN
+F 2 "" H 4100 3250 60  0000 C CNN
+F 3 "" H 4100 3250 60  0000 C CNN
+	1    4100 3250
+	1    0    0    -1
+$EndComp
 $EndSCHEMATC
